File: global.sch (KiCad schematic (older format))
At the start: 37 parts, among them Q5 MMBT3904, U11 74HC165, U12 74HC595, U13 74HC595, U14 74HC595, U5 74HCT125

Commit message: updated footprints
Parts:
- JP1: footprint w_connector:MOLEX_USB_105057 -> w_connector:Kycon_USB_KUSBVLPX-AS1N
Changed lines of the file:
@@
 F 0 "JP1" H 7400 4350 50  0000 L CNN
 F 1 "USB_A" H 7400 4250 50  0000 L CNN
-F 2 "w_connector:MOLEX_USB_105057" H 7750 3850 50  0001 C CNN
+F 2 "w_connector:Kycon_USB_KUSBVLPX-AS1N" H 7750 3850 50  0001 C CNN
 F 3 "http://datasheet.octopart.com/105057-0001-Molex-datasheet-48881000.pdf" H 7750 3850 50  0001 C CNN
 F 4 "Molex" H 7600 3900 60  0001 C CNN "MFN"

Commit message: updated component values and revision
Parts:
- JP1: MFN Molex -> Kycon; MFP 105057-0001 -> KUSBVLPX-AS1N-B
Changed lines of the file:
@@
 Sheet 2 8
 Title "PER|FORMER eurorack sequencer"
-Date "2018-10-09"
-Rev "1.0"
+Date "2019-04-10"
+Rev "1.1"
 Comp "westlicht"
 Comment1 "cc-by-nc-sa"
@@
 F 1 "USB_A" H 7400 4250 50  0000 L CNN
 F 2 "w_connector:Kycon_USB_KUSBVLPX-AS1N" H 7750 3850 50  0001 C CNN
-F 3 "http://datasheet.octopart.com/105057-0001-Molex-datasheet-48881000.pdf" H 7750 3850 50  0001 C CNN
-F 4 "Molex" H 7600 3900 60  0001 C CNN "MFN"
-F 5 "105057-0001" H 7600 3900 60  0001 C CNN "MFP"
+F 3 "https://www.mouser.ch/datasheet/2/222/Kycon_01302017_KUSBVLPX-AS1N-x-1174221.pdf" H 7750 3850 50  0001 C CNN
+F 4 "Kycon" H 7600 3900 60  0001 C CNN "MFN"
+F 5 "KUSBVLPX-AS1N-B" H 7600 3900 60  0001 C CNN "MFP"
 	1    7600 3900
 	1    0    0    -1
@@
 Wire Notes Line
 	600  6400 600  600
+Wire Wire Line
+	4000 3900 4000 4400
+Wire Wire Line
+	4000 2500 4000 3000
+Wire Wire Line
+	4000 1100 4000 1600
+Wire Wire Line
+	2000 5200 2300 5200
+Wire Wire Line
+	1700 5200 2000 5200
+Wire Wire Line
+	2000 5700 2300 5700
+Wire Wire Line
+	1700 5700 2000 5700
+Wire Wire Line
+	5200 5900 5200 6000
+Wire Wire Line
+	5200 6000 5200 6100
+Wire Wire Line
+	2300 5700 2600 5700
+Wire Wire Line
+	2300 5200 2600 5200
+Wire Wire Line
+	1400 5200 1700 5200
+Wire Wire Line
+	1400 5700 1700 5700
+Wire Wire Line
+	3700 2900 3700 4300
+Wire Wire Line
+	3700 4300 3700 5500
+Wire Wire Line
+	3700 1500 4100 1500
+Wire Wire Line
+	3600 2800 3600 4200
+Wire Wire Line
+	3600 1600 3600 2800
+Wire Wire Line
+	9700 4100 9700 4200
+Wire Wire Line
+	9700 4200 9700 4600
+Wire Wire Line
+	9700 4600 9700 4700
+Wire Wire Line
+	9700 4700 9700 4800
+Wire Wire Line
+	9700 4800 9700 4900
+Wire Wire Line
+	9700 4900 9700 5000
+Wire Wire Line
+	9700 5000 9700 5500
+Wire Wire Line
+	9700 5500 9700 5600
+Wire Wire Line
+	9700 5600 9700 5800
+Wire Wire Line
+	7600 4400 7600 4500
+Wire Wire Line
+	5600 4800 5700 4800
+Wire Wire Line
+	5500 4800 5600 4800
+Wire Wire Line
+	5400 4800 5500 4800
+Wire Wire Line
+	5700 4800 6200 4800
+Wire Wire Line
+	5300 5300 5800 5300
+Wire Wire Line
+	5400 5400 5800 5400
+Wire Wire Line
+	5500 5500 5800 5500
+Wire Wire Line
+	5600 5600 5800 5600
+Wire Wire Line
+	5700 5700 5800 5700
+Wire Wire Line
+	1500 1900 1500 2000
+Wire Wire Line
+	1500 1800 1500 1900
+Wire Wire Line
+	1500 1700 1500 1800
+Wire Wire Line
+	1500 1600 1500 1700
+Wire Wire Line
+	4000 6000 4000 6100
+Wire Wire Line
+	4000 5900 4000 6000
+Wire Wire Line
+	8600 1100 8600 1900
+Wire Wire Line
+	8400 1100 8600 1100
+Wire Wire Line
+	8000 1100 8200 1100
+Wire Wire Line
+	8000 2200 8700 2200
+Wire Wire Line
+	8200 1100 8400 1100
+Wire Wire Line
+	8200 1800 8700 1800
+Wire Wire Line
+	8400 1700 8700 1700
+Wire Wire Line
+	8600 2800 8600 2900
+Wire Wire Line
+	9500 5200 9800 5200
+Wire Wire Line
+	9700 5800 9700 5900
+Wire Wire Line
+	3400 2700 3400 4100
+Wire Wire Line
+	2700 2600 2700 2700
+Wire Wire Line
+	3400 2600 3400 2700
+Wire Wire Line
+	2300 2900 2400 2900
+Wire Wire Line
+	2700 3400 2700 3500
 Connection ~ 4000 3900
 Connection ~ 4000 2500
@@
 NoConn ~ 4100 5600
 NoConn ~ 4100 4500
-Wire Wire Line
-	4000 3900 4000 4400
-Wire Wire Line
-	4000 2500 4000 3000
-Wire Wire Line
-	4000 1100 4000 1600
-Wire Wire Line
-	2000 5200 2300 5200
-Wire Wire Line
-	1700 5200 2000 5200
-Wire Wire Line
-	2000 5700 2300 5700
-Wire Wire Line
-	1700 5700 2000 5700
-Wire Wire Line
-	5200 5900 5200 6000
-Wire Wire Line
-	5200 6000 5200 6100
-Wire Wire Line
-	2300 5700 2600 5700
-Wire Wire Line
-	2300 5200 2600 5200
-Wire Wire Line
-	1400 5200 1700 5200
-Wire Wire Line
-	1400 5700 1700 5700
-Wire Wire Line
-	3700 2900 3700 4300
-Wire Wire Line
-	3700 4300 3700 5500
-Wire Wire Line
-	3700 1500 4100 1500
-Wire Wire Line
-	3600 2800 3600 4200
-Wire Wire Line
-	3600 1600 3600 2800
-Wire Wire Line
-	9700 4100 9700 4200
-Wire Wire Line
-	9700 4200 9700 4600
-Wire Wire Line
-	9700 4600 9700 4700
-Wire Wire Line
-	9700 4700 9700 4800
-Wire Wire Line
-	9700 4800 9700 4900
-Wire Wire Line
-	9700 4900 9700 5000
-Wire Wire Line
-	9700 5000 9700 5500
-Wire Wire Line
-	9700 5500 9700 5600
-Wire Wire Line
-	9700 5600 9700 5800
-Wire Wire Line
-	7600 4400 7600 4500
-Wire Wire Line
-	5600 4800 5700 4800
-Wire Wire Line
-	5500 4800 5600 4800
-Wire Wire Line
-	5400 4800 5500 4800
-Wire Wire Line
-	5700 4800 6200 4800
-Wire Wire Line
-	5300 5300 5800 5300
-Wire Wire Line
-	5400 5400 5800 5400
-Wire Wire Line
-	5500 5500 5800 5500
-Wire Wire Line
-	5600 5600 5800 5600
-Wire Wire Line
-	5700 5700 5800 5700
-Wire Wire Line
-	1500 1900 1500 2000
-Wire Wire Line
-	1500 1800 1500 1900
-Wire Wire Line
-	1500 1700 1500 1800
-Wire Wire Line
-	1500 1600 1500 1700
-Wire Wire Line
-	4000 6000 4000 6100
-Wire Wire Line
-	4000 5900 4000 6000
-Wire Wire Line
-	8600 1100 8600 1900
-Wire Wire Line
-	8400 1100 8600 1100
-Wire Wire Line
-	8000 1100 8200 1100
-Wire Wire Line
-	8000 2200 8700 2200
-Wire Wire Line
-	8200 1100 8400 1100
-Wire Wire Line
-	8200 1800 8700 1800
-Wire Wire Line
-	8400 1700 8700 1700
-Wire Wire Line
-	8600 2800 8600 2900
-Wire Wire Line
-	9500 5200 9800 5200
-Wire Wire Line
-	9700 5800 9700 5900
-Wire Wire Line
-	3400 2700 3400 4100
-Wire Wire Line
-	2700 2600 2700 2700
-Wire Wire Line
-	3400 2600 3400 2700
-Wire Wire Line
-	2300 2900 2400 2900
-Wire Wire Line
-	2700 3400 2700 3500
 $EndSCHEMATC

Commit message: add voltage supervisor, add leds to jacks, update footprints
Parts:
- U11, U12, U13, U14: footprint Package_SO:SOIC-16_3.9x9.9mm_P1.27mm -> w_ic:SOIC-16
Changed lines of the file:
@@
 EESchema Schematic File Version 4
-LIBS:sequencer-cache
-EELAYER 26 0
+EELAYER 30 0
 EELAYER END
 $Descr A4 11693 8268
@@
 F 0 "U11" H 4600 4450 60  0000 C CNN
 F 1 "74HC165" H 4600 5450 60  0000 C CNN
-F 2 "Package_SO:SOIC-16_3.9x9.9mm_P1.27mm" H 4100 5300 60  0001 C CNN
+F 2 "w_ic:SOIC-16" H 4100 5300 60  0001 C CNN
 F 3 "https://octopart.com/click/track?ct=datasheets&hlid=24916538&ppid=35776&sid=370&sig=03765d0" H 4100 5300 60  0001 C CNN
 F 4 "Texas Instruments" H 4600 4550 50  0001 C CNN "MFN"
@@
 F 0 "U12" H 4600 250 60  0000 C CNN
 F 1 "74HC595" H 4600 1250 60  0000 C CNN
-F 2 "Package_SO:SOIC-16_3.9x9.9mm_P1.27mm" H 4100 1100 60  0001 C CNN
+F 2 "w_ic:SOIC-16" H 4100 1100 60  0001 C CNN
 F 3 "https://octopart.com/click/track?ct=datasheets&hlid=24917219&ppid=44183&sid=370&sig=036bbbe" H 4100 1100 60  0001 C CNN
 F 4 "Texas Instruments" H 4600 350 50  0001 C CNN "MFN"
@@
 F 0 "U13" H 4600 1650 60  0000 C CNN
 F 1 "74HC595" H 4600 2650 60  0000 C CNN
-F 2 "Package_SO:SOIC-16_3.9x9.9mm_P1.27mm" H 4100 2500 60  0001 C CNN
+F 2 "w_ic:SOIC-16" H 4100 2500 60  0001 C CNN
 F 3 "https://octopart.com/click/track?ct=datasheets&hlid=24917219&ppid=44183&sid=370&sig=036bbbe" H 4100 2500 60  0001 C CNN
 F 4 "Texas Instruments" H 4600 1750 50  0001 C CNN "MFN"
@@
 F 0 "U14" H 4600 3050 60  0000 C CNN
 F 1 "74HC595" H 4600 4050 60  0000 C CNN
-F 2 "Package_SO:SOIC-16_3.9x9.9mm_P1.27mm" H 4100 3900 60  0001 C CNN
+F 2 "w_ic:SOIC-16" H 4100 3900 60  0001 C CNN
 F 3 "https://octopart.com/click/track?ct=datasheets&hlid=24917219&ppid=44183&sid=370&sig=036bbbe" H 4100 3900 60  0001 C CNN
 F 4 "Texas Instruments" H 4600 3150 50  0001 C CNN "MFN"
