File: power.sch (KiCad schematic (older format))
At the start: 24 parts, among them U10 LM1117-3.3, U16 R-78E5.0-1.0, U3 STMPS2151, U7 LM1117-3.3

Commit message: small changes
Parts:
- U3: footprint Package_TO_SOT_SMD:SOT-23-5 -> Package_SO:TSSOP-8_4.4x3mm_P0.65mm
Changed lines of the file:
@@
 F 0 "U3" H 2100 3300 50  0000 C CNN
 F 1 "STMPS2151" H 2100 2900 50  0000 C CNN
-F 2 "Package_TO_SOT_SMD:SOT-23-5" H 2100 3100 60  0001 C CNN
+F 2 "Package_SO:TSSOP-8_4.4x3mm_P0.65mm" H 2100 3100 60  0001 C CNN
 F 3 "http://datasheet.octopart.com/STMPS2151STR-STMicroelectronics-datasheet-15207125.pdf" H 2100 3100 60  0001 C CNN
 F 4 "STMicroelectronics" H 2100 3100 60  0001 C CNN "MFN"
@@
 Connection ~ 2000 1300
 Connection ~ 2000 1700
+Text GLabel 2400 3500 2    51   Output ~ 0
+USB_5V
+Text GLabel 2400 3650 2    51   Output ~ 0
+USB_5V
+$Comp
+L power:+5V #PWR0162
+U 1 1 5F56DEF5
+P 1800 3500
+F 0 "#PWR0162" H 1800 3350 50  0001 C CNN
+F 1 "+5V" H 1800 3640 50  0000 C CNN
+F 2 "" H 1800 3500 50  0001 C CNN
+F 3 "" H 1800 3500 50  0001 C CNN
+	1    1800 3500
+	1    0    0    -1
+$EndComp
 $EndSCHEMATC
